File: hardware/boards/mini/v0.2/mini_v0.2.kicad_sch (KiCad schematic)
At the start: 99 parts, among them IC1 NAU88C22YG, IC3 IS42S16160J-6BLI, J2 Top, J3 Bottom, Q1 PMV37EN22, U1 W25Q128JVP, U2 LTV-217-G, U4 STM32H750XBHx, Y1 Crystal_GND24, Y3 32.768kHz

Commit message: mini: resolve ERC errors
Connections:
- net BOOT0: now also J2.25
- no-connect marks 3 -> 95
Other:
- note added: "Reverse voltage and short circuit protection circuit"
- note removed: "Reverse voltage protection circuit"
