File: hardware/boards/card/v0.1/codec.kicad_sch (KiCad schematic)
At the start: 0 parts

Commit message: card: add filter caps for codec
Parts:
- added C15, C26: 2n7 C0G, rhais_rcl.pretty-main:C0402, symbol Device:C_Small
- added C16, C17, C23, C25: 470pF C0G, rhais_rcl.pretty-main:C0402, symbol Device:C_Small
- added C20, C22: 0.1uF X7R, rhais_rcl.pretty-main:C0402, symbol Device:C_Small
- added C21, C29: 4.7uF X7R, rhais_rcl.pretty-main:C0402, symbol Device:C_Small
- added C27, C28: 2n2 FILM, rhais_rcl.pretty-main:C0603, symbol Device:C_Small
- added C79: 8200pF X5R, rhais_rcl.pretty-main:C0402, symbol Device:C_Small
- added C80: 220pF X5R, rhais_rcl.pretty-main:C0402, symbol Device:C_Small
- added C81, C83: 0.1uF X5R, rhais_rcl.pretty-main:C0402, symbol Device:C_Small
- added C82: 4.7uF X5R, rhais_rcl.pretty-main:C0402, symbol Device:C_Small
- added C84: 100uF X5R, rhais_rcl.pretty-main:C0402, symbol Device:C_Small
- added J8: Conn_01x16_Pin, Connector_PinHeader_1.27mm:PinHeader_1x16_P1.27mm_Vertical, symbol Connector:Conn_01x16_Pin
- added J9: AUDIO_IN, Connector_PinHeader_1.27mm:PinHeader_1x02_P1.27mm_Vertical, symbol Connector:Conn_01x02_Pin
- added R1, R18, R20, R4: 91R, rhais_rcl.pretty-main:R0402, symbol Device:R
- added R10, R14: 3.32k, rhais_rcl.pretty-main:R0402, symbol Device:R_Small
- added R11, R12: 10k, rhais_rcl.pretty-main:R0402, symbol Device:R_Small
- added R13, R9: 2.8k, rhais_rcl.pretty-main:R0402, symbol Device:R_Small
- added R15, R17, R19, R2, R3, R5: 634R, rhais_rcl.pretty-main:R0402, symbol Device:R
- added R16, R6: 332R, rhais_rcl.pretty-main:R0402, symbol Device:R
- added R7, R8, R85, R86: 10k, rhais_rcl.pretty-main:R0402, symbol Device:R
- added R87: 1.6k, rhais_rcl.pretty-main:R0402, symbol Device:R_Small
- added U1: CS42528K-CQZ, Package_QFP:LQFP-64_10x10mm_P0.5mm, symbol Northernpaws_Audio:CS42528K-CQZ
- added U3, U4: NJM4580E-TE1, Package_SO:TSSOP-8_3x3mm_P0.65mm, symbol Amplifier_Operational:NJM4580
Connections:
- new net: C16.2, R1.1, U3.7
- new net: C25.2, R20.1, U4.7
- new net: C20.1, C21.1, R10.1, R6.1, R7.1, R9.2
- new net: C83.1, C84.1, U1.18 (FILT+)
- new net: C17.2, R3.1, R4.1, U3.1
- new net: C16.1, R2.1, R3.2, U3.6 (-)
- new net: C17.1, R5.1, U3.2 (-)
- new net: R86.1, U1.9 (AD1/CDIN)
- new net: C80.1, R87.1, U1.39 (LPFLT)
- new net: C79.1, R87.2
- new net: C22.1, C29.1, R13.2, R14.1, R16.1, R8.1
- new net: C23.2, R17.1, R18.1, U4.1
- new net: C25.1, R17.2, R19.1, U4.6 (-)
- new net: C23.1, R15.1, U4.2 (-)
- new net: C28.2, R8.2, U4.3 (+)
- new net: R6.2, U3.5 (+)
- new net: R16.2, U4.5 (+)
- new net: C27.2, R7.2, U3.3 (+)
- new net: R85.1, U1.10 (AD0/CS)
- new net: C81.1, C82.1, U1.17 (VQ)
- new net +3.3V: U1.4 (VD), U1.51 (VD), U1.53 (VLS), U1.6 (VLC)
- new net +5V: R13.1, R9.1, U1.24 (VA), U1.41 (VA), U3.8 (V+), U4.4 (V-)
- new net AINL+: C15.1, R4.2, R5.2, U1.15 (AINL+)
- new net AINL-: C15.2, R1.2, R2.2, U1.16 (AINL-)
- new net AINR+: C26.1, R15.2, R18.2, U1.14 (AINR+)
- new net AINR-: C26.2, R19.2, R20.2, U1.13 (AINR-)
- new net AOUTA1+: U1.36 (AOUTA1+)
- new net AOUTA1-: U1.37 (AOUTA1-)
- new net AOUTA2+: U1.32 (AOUTA2+)
- new net AOUTA2-: U1.33 (AOUTA2-)
- new net AOUTA3+: U1.28 (AOUTA3+)
- new net AOUTA3-: U1.29 (AOUTA3-)
- new net AOUTA4+: U1.22 (AOUTA4+)
- new net AOUTA4-: U1.23 (AOUTA4-)
- new net AOUTB1+: U1.35 (AOUTB1+)
- new net AOUTB1-: U1.34 (AOUTB1-)
- new net AOUTB2+: U1.31 (AOUTB2+)
- new net AOUTB2-: U1.30 (AOUTB2-)
- new net AOUTB3+: U1.27 (AOUTB3+)
- new net AOUTB3-: U1.26 (AOUTB3-)
- new net AOUTB4+: U1.21 (AOUTB4+)
- new net AOUTB4-: U1.20 (AOUTB4-)
- new net GND: C20.2, C21.2, C22.2, C29.2, C79.2, C80.2, C81.2, C82.2, C83.2, C84.2, R10.2, R11.2, R12.2, R14.2, R85.2, R86.2, U1.19 (REFGND), U1.25 (AGND), U1.40 (AGND), U1.5 (DGND), U1.52 (DGND), U3.4 (V-), U4.8 (V+)
- new net I2C2_SCL: U1.7 (SCL/CCLK)
- new net I2C2_SDA: U1.8 (SDA/CDOUT)
- new net IN_L: C27.1, J9.1 (Pin_1), R11.1
- new net IN_R: C28.1, J9.2 (Pin_2), R12.1
- new net OUT_A1: J8.11 (Pin_11)
- new net OUT_A2: J8.8 (Pin_8)
- new net OUT_A3: J8.5 (Pin_5)
- new net OUT_A4: J8.2 (Pin_2)
- new net OUT_B1: J8.10 (Pin_10)
- new net OUT_B2: J8.7 (Pin_7)
- new net OUT_B3: J8.4 (Pin_4)
- new net OUT_B4: J8.1 (Pin_1)
- new net SAI1_FS_A: U1.3 (CX_LRCK)
- new net SAI1_MCLK_A: U1.59 (OMCK)
- new net SAI1_SCK_A: U1.2 (CX_SCLK)
- new net SAI1_SD_A: U1.63 (CX_SDIN3)
- new net SAI1_SD_B: U1.62 (CX_SDIN4)
- new net SAI2_SD_A: U1.1 (CX_SDIN1)
- new net SAI2_SD_B: U1.64 (CX_SDIN2)
- new net SAI4_SD_B: U1.56 (CX_SDOUT)
- no-connect marks 0 -> 12
Other:
- added sheet Codec Output Stage 1 (codec_output_stage.kicad_sch)
- added sheet Codec Output Stage 2 (codec_output_stage.kicad_sch)
- added sheet Codec Output Stage 3 (codec_output_stage.kicad_sch)
- added sheet Codec Output Stage 4 (codec_output_stage.kicad_sch)
- note added: "+2.7v"
- note added: "3MHz Band Limiting Metal foil (or thin-film) resistors"
- note added: "AD0 connected through resistor to HIGH or LOW signals I2C mode."
- note added: "Line-level differential analog inputs, must be externally biased to VQ, approximately 2.7 V, before being applied to these inputs."
- note added: "One-Line Mode Config #1 for CS42528K-CQZ @ 48kHz"
- note added: "The LRCLK must be equal to the sample rate, Fs, and must be derived from the supplied master clock, OMCK, or the output of the PLL. The serial bit clock, CX_SCLK, must be synchronously derived from the master clock and be equal to 128x, 64x, 48x or 32x Fs, depending on the interface format selected and desired speed mode."
- note added: "Unfortunately the analog path requires +5V and will not function on +3.3v."
- note added: "https://statics.cirrus.com/pubs/rdDatasheet/CRD42528-2.pdf"
- note added: "line-level differential outputs biased to a DC level of VQ."
