File: hardware/boards/card/v0.1/codec_output_stage.kicad_sch (KiCad schematic)
At the start: 29 parts, among them U5 NJM4580E-TE1

Commit message: card: route remaining 2 codec output stages
Parts:
- added C75: 100nF X5R, rhais_rcl.pretty-main:C0402, symbol Device:C_Small
Connections:
- net GND: now also U5.8 (V+), C75.2
- new net +5V: C75.1, U5.4 (V-)

Commit message: card: add filter caps for codec
Parts:
- added unit 3 of U8
- renumbered C18 to C63, C19 to C64, C33 to C65, C34 to C66, C30 to C67, C35 to C68, C31 to C69, C36 to C70, C24 to C71, C37 to C72, C32 to C73, C38 to C74, C75 to C78, R22 to R69, R23 to R70, R29 to R71, R30 to R72, R25 to R73, R21 to R74, R24 to R75, R26 to R76, R31 to R77, R32 to R78, R33 to R79, R34 to R80, R27 to R81, R35 to R82, R28 to R83, R36 to R84, U5 to U8
Connections:
- net +5V: now also U8.4 (V-); no longer U8.4 (V-)
- net GND: now also U8.8 (V+); no longer U8.8 (V+)
